File: ESPLED.kicad_pcb (KiCad board)
At the start: 2 copper layers, 83.8 x 43.2 mm, 20 parts, among them CON1 BARREL_JACK, P1 PROG, P2 LED_CON, P3 LED_CON_SCREW, P4 LED_CON_SCREW, Q1 IRLZ34N, Q2 IRLZ34N, Q3 IRLZ34N, SW1 Reset, U1 AP7333, U2 ESP-07v2

Commit message: All coponents set
Parts:
- U1: value AP7333 -> LM1117-3.3
Connections:
- Q2 pad 1: Net-(P2-Pad2) -> Net-(Q2-Pad1)
- Q2 pad 2: Net-(Q2-Pad2) -> Net-(P2-Pad2)
- R2 pad 1: Net-(Q2-Pad2) -> Net-(Q2-Pad1)
- U1 pad 1: +12V -> GND
- U1 pad 3: GND -> +12V
Routing:
- net Net-(P2-Pad3): track 96.9 -> 31.2 mm
- net Net-(Q2-Pad1): track 0.00 -> 52.4 mm
- net Net-(P2-Pad2): track 71.6 -> 31.6 mm
- net Net-(Q3-Pad2): track 32.0 -> 0.00 mm
- net Net-(Q2-Pad2): track 12.4 -> 0.00 mm
- net GND: track 17.1 -> 16.1 mm, vias 1 -> 0
- net +12V: track 47.4 -> 48.4 mm, vias 0 -> 1
