File: ESPLED.kicad_pcb (KiCad board)
At the start: 2 copper layers, 100 x 50 mm, 43 parts, among them CON1 BARREL_JACK, J1 USB_B_Micro, J2 LED_CON_RGB, J3 LED_CON_WW, J4 MIC, P1 LED_CON_SCREW, P2 LED_CON_SCREW, P3 LED_CON_SCREW, Q1 IRLZ34N, Q2 IRLZ34N, Q3 IRLZ34N, Q4 IRLZ34N, Q5 IRLZ34N, SW1 Reset, SW2 Program, SW3 Mode, U1 AMS1117-3.3, U2 ESP-07v2, U3 INTERFACE-CH340G, U4 DS18B20, Y1 Crystal

Commit message: Routed
Parts:
- added C8: 100nF, Capacitor_SMD:C_0603_1608Metric_Pad1.05x0.95mm_HandSolder, F.Cu at (167.1, 100.6)
- added C9: 100nF, Capacitor_SMD:C_0603_1608Metric_Pad1.05x0.95mm_HandSolder, F.Cu at (159.7, 91.9)
- added JP10: GPIO LINK, Jumper:SolderJumper-2_P1.3mm_Open_RoundedPad1.0x1.5mm, F.Cu at (161.0, 95.0)
- added JP6: GPIO LINK, Jumper:SolderJumper-2_P1.3mm_Open_RoundedPad1.0x1.5mm, F.Cu at (169.2, 95.0)
- added JP7: GPIO LINK, Jumper:SolderJumper-2_P1.3mm_Open_RoundedPad1.0x1.5mm, F.Cu at (167.1, 95.0)
- added JP8: GPIO LINK, Jumper:SolderJumper-2_P1.3mm_Open_RoundedPad1.0x1.5mm, F.Cu at (165.1, 95.0)
- added JP9: GPIO LINK, Jumper:SolderJumper-2_P1.3mm_Open_RoundedPad1.0x1.5mm, F.Cu at (163.1, 95.0)
- added U5: TXS0108EPW, Package_SO:TSSOP-20_4.4x6.5mm_P0.65mm, F.Cu at (164.8, 95.0)
- U3: footprint Package_SO:SOIC-16W_5.3x10.2mm_P1.27mm -> Package_SO:SOP-16_4.4x10.4mm_P1.27mm
- moved R6 4.95 mm to (155.2, 87.3), turned to 90 degrees
- moved R7 2.16 mm to (177.5, 87.2)
- moved P1 2.09 mm to (185.5, 76.0)
- moved U2 1.99 mm to (167.0, 79.0)
- moved P3 1.72 mm to (185.5, 96.4)
- moved J1 1.38 mm to (96.0, 71.1)
- moved P2 0.52 mm to (185.5, 86.2)
- moved U3 0.40 mm to (124.6, 81.8)
Connections:
- JP1 pad 2: Net-(JP1-Pad2) -> HSIG1
- JP2 pad 2: Net-(JP2-Pad2) -> HSIG2
- JP3 pad 2: Net-(JP3-Pad2) -> HSIG3
- JP4 pad 2: Net-(JP4-Pad2) -> HSIG4
- JP5 pad 2: Net-(JP5-Pad2) -> HSIG5
- R1 pad 2: Net-(JP1-Pad2) -> HSIG1
- R2 pad 2: Net-(JP2-Pad2) -> HSIG2
- R3 pad 2: Net-(JP3-Pad2) -> HSIG3
- R4 pad 2: Net-(JP4-Pad2) -> HSIG4
- R5 pad 2: Net-(JP5-Pad2) -> HSIG5
- U2 pad 14: Net-(JP5-Pad2) -> SIG1
- U2 pad 4: Net-(JP1-Pad2) -> SIG2
- U2 pad 5: Net-(JP2-Pad2) -> SIG3
- U2 pad 6: Net-(JP3-Pad2) -> SIG4
- U2 pad 7: Net-(JP4-Pad2) -> SIG5
Routing:
- net HSIG1: track 0.00 -> 85.7 mm
- net HSIG2: track 0.00 -> 70.6 mm
- net Net-(JP1-Pad2): track 68.7 -> 0.00 mm
- net HSIG3: track 0.00 -> 56.8 mm
- net Net-(JP2-Pad2): track 56.3 -> 0.00 mm
- net HSIG4: track 0.00 -> 43.6 mm
- net Net-(JP5-Pad2): track 43.0 -> 0.00 mm
- net Net-(JP3-Pad2): track 42.7 -> 0.00 mm
- net HSIG5: track 0.00 -> 31.0 mm
- net +12V: track 173.8 -> 203.0 mm, vias 0 -> 1
- net Net-(JP4-Pad2): track 29.1 -> 0.00 mm
- net +3V3: track 69.7 -> 97.0 mm, vias 1 -> 2
- net SIG1: track 0.00 -> 24.6 mm, vias 0 -> 2
- net SIG2: track 0.00 -> 18.6 mm
- net SIG3: track 0.00 -> 15.7 mm
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