File: ESPLED.kicad_pcb (KiCad board)
At the start: 2 copper layers, 100 x 50 mm, 51 parts, among them CON1 BARREL_JACK, J1 USB, J2 LED_CON_RGB, J3 LED_CON_WW, J4 MIC, P1 LED_CON_SCREW, P2 LED_CON_SCREW, P3 LED_CON_SCREW, Q1 IRLZ34N, Q2 IRLZ34N, Q3 IRLZ34N, Q4 IRLZ34N, Q5 IRLZ34N, SW1 Reset, SW2 Program, SW3 Mode, U1 AMS1117-3.3, U2 ESP-07v2, U3 CH340G, U4 DS18B20, U5 TXS0108EPW, Y1 12MHz

Commit message: final 01:11
Parts:
- added G***: LOGO, icons:github-espled12, B.Cu at (173.9, 87.0)
- U2: value ESP-07v2 -> ESP8266-12F
Other:
- board text added: "+12V/+5V"
- board text added: "CH1"
- board text added: "CH2"
- board text added: "CH3"
- board text added: "CH4"
- board text added: "CH5"
- board text added: "espled Rev 1.0 16.01.2019 Andre & Dominik"
- board text added: "github.com/Yottabits/espled"
- board text removed: "Ĉ WG Guys"
