File: hardware/ESPLED.sch (KiCad schematic (older format))
At the start: 51 parts, among them CON1 BARREL_JACK, J1 USB_B_Micro, J2 LED_CON_RGB, J3 LED_CON_WW, J4 MIC, P1 LED_CON_SCREW, P2 LED_CON_SCREW, P3 LED_CON_SCREW, Q1 IRLZ34N, Q2 IRLZ34N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

Commit message: Change Capacitor size, fix #23 move C4 near ESP8266, fix #11 change label P1 to P3, fix #12
Parts:
- C2: value 1000uF -> 22uF
- renumbered P3 to P1, P1 to P3
Changed lines of the file:
@@
 P 4200 7100
 F 0 "C2" H 4225 7200 50  0000 L CNN
-F 1 "1000uF" H 4225 7000 50  0000 L CNN
+F 1 "22uF" H 4225 7000 50  0000 L CNN
 F 2 "Capacitor_SMD:CP_Elec_10x10.5" H 4238 6950 50  0001 C CNN
 F 3 "" H 4200 7100 50  0000 C CNN
@@
 $EndComp
 $Comp
-L ESPLED-rescue:SCREW-TERMINAL-GREEN_2P-3.5_ P3
+L ESPLED-rescue:SCREW-TERMINAL-GREEN_2P-3.5_ P1
 U 1 1 5A986FD8
 P 1550 1450
-F 0 "P3" H 1700 1450 45  0000 L BNN
+F 0 "P1" H 1700 1450 45  0000 L BNN
 F 1 "LED_CON_SCREW" H 850 1450 45  0000 L BNN
 F 2 "TerminalBlock:TerminalBlock_Altech_AK300-2_P5.00mm" H 1550 1450 60  0001 C CNN
@@
 $EndComp
 $Comp
-L ESPLED-rescue:SCREW-TERMINAL-GREEN_2P-3.5_ P1
+L ESPLED-rescue:SCREW-TERMINAL-GREEN_2P-3.5_ P3
 U 1 1 5A987158
 P 2700 1450
-F 0 "P1" H 2850 1450 45  0000 L BNN
+F 0 "P3" H 2850 1450 45  0000 L BNN
 F 1 "LED_CON_SCREW" H 2000 1450 45  0000 L BNN
 F 2 "TerminalBlock:TerminalBlock_Altech_AK300-2_P5.00mm" H 2700 1450 60  0001 C CNN
